Commit message: [shm_transport] add usb camera shm transport

File: src/test11_description/urdf/test11.xacro (robot description, xacro)
@@ -145,5 +145,5 @@
 </joint>
 <joint name="j4" type="fixed">
-  <origin xyz="0.162817 0.0 0.060341" rpy="0 0 1.5708"/>
+  <origin xyz="0.162817 0.0 0.060341" rpy="0 0 -1.5708"/>
   <parent link="base_link"/>
   <child link="laser_link"/>
